File: S-100-Template.kicad_pcb (KiCad board)
At the start: 2 copper layers, 254 x 134.6 mm, 3 parts, among them J1 S100

Commit message: Add image & rescue cruft
Other:
- board text added: "-"
- board text added: "1"
- board text added: "10"
- board text added: "100"
- board text added: "20"
- board text added: "30"
- board text added: "40"
- board text added: "50"
- board text added: "51"
- board text added: "60"
- board text added: "70"
- board text added: "80"
- board text added: "90"
Changed lines of the file:
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@@
   (general
     (thickness 1.6)
-    (drawings 25)
+    (drawings 47)
     (tracks 0)
     (zones 0)
@@
       (solder_mask_margin 1.27))
   )
+  (gr_text - (at 79.756 150.622) (layer B.SilkS)
+    (effects (font (size 1 1) (thickness 0.15)))
+  )
+  (gr_text - (at 111.506 150.622) (layer B.SilkS)
+    (effects (font (size 1 1) (thickness 0.15)))
+  )
+  (gr_text - (at 143.256 150.622) (layer B.SilkS)
+    (effects (font (size 1 1) (thickness 0.15)))
+  )
+  (gr_text - (at 175.006 150.622) (layer B.SilkS)
+    (effects (font (size 1 1) (thickness 0.15)))
+  )
+  (gr_text - (at 206.756 150.622) (layer B.SilkS)
+    (effects (font (size 1 1) (thickness 0.15)))
+  )
+  (gr_text - (at 206.756 150.622) (layer F.SilkS)
+    (effects (font (size 1 1) (thickness 0.15)))
+  )
+  (gr_text - (at 175.006 150.622) (layer F.SilkS)
+    (effects (font (size 1 1) (thickness 0.15)))
+  )
+  (gr_text - (at 143.256 150.622) (layer F.SilkS)
+    (effects (font (size 1 1) (thickness 0.15)))
+  )
+  (gr_text - (at 111.506 150.622) (layer F.SilkS)
+    (effects (font (size 1 1) (thickness 0.15)))
+  )
+  (gr_text - (at 79.756 150.622) (layer F.SilkS)
+    (effects (font (size 1 1) (thickness 0.15)))
+  )
+  (gr_text 100 (at 223.012 150.368) (layer B.SilkS)
+    (effects (font (size 1 1) (thickness 0.15)) (justify mirror))
+  )
+  (gr_text 90 (at 190.754 150.368) (layer B.SilkS)
+    (effects (font (size 1 1) (thickness 0.15)) (justify mirror))
+  )
+  (gr_text 80 (at 159.004 150.368) (layer B.SilkS)
+    (effects (font (size 1 1) (thickness 0.15)) (justify mirror))
+  )
+  (gr_text 70 (at 127.254 150.368) (layer B.SilkS)
+    (effects (font (size 1 1) (thickness 0.15)) (justify mirror))
+  )
+  (gr_text 60 (at 95.504 150.368) (layer B.SilkS)
+    (effects (font (size 1 1) (thickness 0.15)) (justify mirror))
+  )
+  (gr_text 51 (at 66.548 150.368) (layer B.SilkS)
+    (effects (font (size 1 1) (thickness 0.15)) (justify mirror))
+  )
+  (gr_text 50 (at 223.012 150.368) (layer F.SilkS)
+    (effects (font (size 1 1) (thickness 0.15)))
+  )
+  (gr_text 40 (at 190.754 150.368) (layer F.SilkS)
+    (effects (font (size 1 1) (thickness 0.15)))
+  )
+  (gr_text 30 (at 159.004 150.368) (layer F.SilkS)
+    (effects (font (size 1 1) (thickness 0.15)))
+  )
+  (gr_text 20 (at 127.254 150.368) (layer F.SilkS)
+    (effects (font (size 1 1) (thickness 0.15)))
+  )
+  (gr_text 10 (at 95.504 150.368) (layer F.SilkS)
+    (effects (font (size 1 1) (thickness 0.15)))
+  )
+  (gr_text 1 (at 66.548 150.368) (layer F.SilkS)
+    (effects (font (size 1 1) (thickness 0.15)))
+  )
   (gr_arc (start 225.933 152.908) (end 225.933 152.4) (angle -90) (layer Edge.Cuts) (width 0.3))

Commit message: Re-implement from scratch in kicad 9
Parts:
- H1, H2: value Ejector -> MountingHole; footprint jb-footprint:MountingHole_2.7mm_M2.5 -> MountingHole:MountingHole_2.5mm
- J1: value S100 -> ~; footprint jb-footprint:S100_MALE -> S100-footprints:S100-Edge-Connector
- moved J1 74.7 mm to (138.4, 158.8)
- moved H2 6.35 mm to (266.7, 31.8)
- moved H1 6.35 mm to (25.4, 31.8)
Connections:
- J1 pad 1: Net-(J1-Pad1) -> unconnected-(J1-+8-Pad1)
- J1 pad 10: Net-(J1-Pad10) -> unconnected-(J1-~{VI6}-Pad10)
- J1 pad 100: Net-(J1-Pad100) -> unconnected-(J1-GND-Pad100)
- J1 pad 11: Net-(J1-Pad11) -> unconnected-(J1-~{VI7}-Pad11)
- J1 pad 12: Net-(J1-Pad12) -> unconnected-(J1-~{NMI}-Pad12)
- J1 pad 13: Net-(J1-Pad13) -> unconnected-(J1-~{PWRFAIL}-Pad13)
- J1 pad 14: Net-(J1-Pad14) -> unconnected-(J1-~{DMA3}-Pad14)
- J1 pad 15: Net-(J1-Pad15) -> unconnected-(J1-A18-Pad15)
- J1 pad 16: Net-(J1-Pad16) -> unconnected-(J1-A16-Pad16)
- J1 pad 17: Net-(J1-Pad17) -> unconnected-(J1-A17-Pad17)
- J1 pad 18: Net-(J1-Pad18) -> unconnected-(J1-~{SDSB}-Pad18)
- J1 pad 19: Net-(J1-Pad19) -> unconnected-(J1-~{CDSB}-Pad19)
- J1 pad 2: Net-(J1-Pad2) -> unconnected-(J1-+16-Pad2)
- J1 pad 20: Net-(J1-Pad20) -> unconnected-(J1-GND-Pad20)
- J1 pad 21: Net-(J1-Pad21) -> unconnected-(J1-NDEF-Pad21)
- J1 pad 22: Net-(J1-Pad22) -> unconnected-(J1-~{ADBB}-Pad22)
- J1 pad 23: Net-(J1-Pad23) -> unconnected-(J1-~{DODSB}-Pad23)
- J1 pad 24: Net-(J1-Pad24) -> unconnected-(J1-PHI-Pad24)
- J1 pad 25: Net-(J1-Pad25) -> unconnected-(J1-~{pSTVAL}-Pad25)
- J1 pad 26: Net-(J1-Pad26) -> unconnected-(J1-pHLDA-Pad26)
- J1 pad 27: Net-(J1-Pad27) -> unconnected-(J1-RFU-Pad27)
- J1 pad 28: Net-(J1-Pad28) -> unconnected-(J1-RFU-Pad28)
- J1 pad 29: Net-(J1-Pad29) -> unconnected-(J1-A5-Pad29)
- J1 pad 3: Net-(J1-Pad3) -> unconnected-(J1-XRDY-Pad3)
- J1 pad 30: Net-(J1-Pad30) -> unconnected-(J1-A4-Pad30)
- J1 pad 31: Net-(J1-Pad31) -> unconnected-(J1-A3-Pad31)
- J1 pad 32: Net-(J1-Pad32) -> unconnected-(J1-A15-Pad32)
- J1 pad 33: Net-(J1-Pad33) -> unconnected-(J1-A12-Pad33)
- J1 pad 34: Net-(J1-Pad34) -> unconnected-(J1-A9-Pad34)
- J1 pad 35: Net-(J1-Pad35) -> unconnected-(J1-DO1-Pad35)
- J1 pad 36: Net-(J1-Pad36) -> unconnected-(J1-DO0-Pad36)
- J1 pad 37: Net-(J1-Pad37) -> unconnected-(J1-A10-Pad37)
- J1 pad 38: Net-(J1-Pad38) -> unconnected-(J1-DO4-Pad38)
- J1 pad 39: Net-(J1-Pad39) -> unconnected-(J1-DO5-Pad39)
- J1 pad 4: Net-(J1-Pad4) -> unconnected-(J1-~{VI0}-Pad4)
- J1 pad 40: Net-(J1-Pad40) -> unconnected-(J1-DO6-Pad40)
- J1 pad 41: Net-(J1-Pad41) -> unconnected-(J1-DI2-Pad41)
- J1 pad 42: Net-(J1-Pad42) -> unconnected-(J1-DI3-Pad42)
- J1 pad 43: Net-(J1-Pad43) -> unconnected-(J1-DI7-Pad43)
- J1 pad 44: Net-(J1-Pad44) -> unconnected-(J1-sM1-Pad44)
- J1 pad 45: Net-(J1-Pad45) -> unconnected-(J1-sOUT-Pad45)
- J1 pad 46: Net-(J1-Pad46) -> unconnected-(J1-sINP-Pad46)
- J1 pad 47: Net-(J1-Pad47) -> unconnected-(J1-sMEMR-Pad47)
- J1 pad 48: Net-(J1-Pad48) -> unconnected-(J1-sHLTA-Pad48)
- J1 pad 49: Net-(J1-Pad49) -> unconnected-(J1-CLOCK-Pad49)
- J1 pad 5: Net-(J1-Pad5) -> unconnected-(J1-~{VI1}-Pad5)
- J1 pad 50: Net-(J1-Pad50) -> unconnected-(J1-GND-Pad50)
- J1 pad 51: Net-(J1-Pad51) -> unconnected-(J1-+8-Pad51)
- J1 pad 52: Net-(J1-Pad52) -> unconnected-(J1--16-Pad52)
- J1 pad 53: Net-(J1-Pad53) -> unconnected-(J1-GND-Pad53)
- J1 pad 54: Net-(J1-Pad54) -> unconnected-(J1-~{SLV_CLR}-Pad54)
- J1 pad 55: Net-(J1-Pad55) -> unconnected-(J1-~{DMA0}-Pad55)
- J1 pad 56: Net-(J1-Pad56) -> unconnected-(J1-~{DMA1}-Pad56)
- J1 pad 57: Net-(J1-Pad57) -> unconnected-(J1-~{DMA2}-Pad57)
- J1 pad 58: Net-(J1-Pad58) -> unconnected-(J1-~{sXTRQ}-Pad58)
- J1 pad 59: Net-(J1-Pad59) -> unconnected-(J1-A19-Pad59)
- J1 pad 6: Net-(J1-Pad6) -> unconnected-(J1-~{VI2}-Pad6)
- J1 pad 60: Net-(J1-Pad60) -> unconnected-(J1-~{SIXTN}-Pad60)
- J1 pad 61: Net-(J1-Pad61) -> unconnected-(J1-A20-Pad61)
- J1 pad 62: Net-(J1-Pad62) -> unconnected-(J1-A21-Pad62)
- J1 pad 63: Net-(J1-Pad63) -> unconnected-(J1-A22-Pad63)
- J1 pad 64: Net-(J1-Pad64) -> unconnected-(J1-A23-Pad64)
- J1 pad 65: Net-(J1-Pad65) -> unconnected-(J1-NDEF-Pad65)
- J1 pad 66: Net-(J1-Pad66) -> unconnected-(J1-NDEF-Pad66)
- J1 pad 67: Net-(J1-Pad67) -> unconnected-(J1-~{PHANTOM}-Pad67)
- J1 pad 68: Net-(J1-Pad68) -> unconnected-(J1-MWRT-Pad68)
- J1 pad 69: Net-(J1-Pad69) -> unconnected-(J1-RFU-Pad69)
- J1 pad 7: Net-(J1-Pad7) -> unconnected-(J1-~{VI3}-Pad7)
- J1 pad 70: Net-(J1-Pad70) -> unconnected-(J1-GND-Pad70)
- J1 pad 71: Net-(J1-Pad71) -> unconnected-(J1-RFU-Pad71)
- J1 pad 72: Net-(J1-Pad72) -> unconnected-(J1-RDY-Pad72)
- J1 pad 73: Net-(J1-Pad73) -> unconnected-(J1-~{INT}-Pad73)
- J1 pad 74: Net-(J1-Pad74) -> unconnected-(J1-~{HOLD}-Pad74)
- J1 pad 75: Net-(J1-Pad75) -> unconnected-(J1-~{RESET}-Pad75)
- J1 pad 76: Net-(J1-Pad76) -> unconnected-(J1-pSYNC-Pad76)
- J1 pad 77: Net-(J1-Pad77) -> unconnected-(J1-~{pWR}-Pad77)
- J1 pad 78: Net-(J1-Pad78) -> unconnected-(J1-pDBIN-Pad78)
- J1 pad 79: Net-(J1-Pad79) -> unconnected-(J1-A0-Pad79)
- J1 pad 8: Net-(J1-Pad8) -> unconnected-(J1-~{VI4}-Pad8)
- J1 pad 80: Net-(J1-Pad80) -> unconnected-(J1-A1-Pad80)
- J1 pad 81: Net-(J1-Pad81) -> unconnected-(J1-A2-Pad81)
- J1 pad 82: Net-(J1-Pad82) -> unconnected-(J1-A6-Pad82)
- J1 pad 83: Net-(J1-Pad83) -> unconnected-(J1-A7-Pad83)
- J1 pad 84: Net-(J1-Pad84) -> unconnected-(J1-A8-Pad84)
- J1 pad 85: Net-(J1-Pad85) -> unconnected-(J1-A13-Pad85)
- J1 pad 86: Net-(J1-Pad86) -> unconnected-(J1-A14-Pad86)
- J1 pad 87: Net-(J1-Pad87) -> unconnected-(J1-A11-Pad87)
- J1 pad 88: Net-(J1-Pad88) -> unconnected-(J1-DO2-Pad88)
- J1 pad 89: Net-(J1-Pad89) -> unconnected-(J1-DO3-Pad89)
- J1 pad 9: Net-(J1-Pad9) -> unconnected-(J1-~{VI5}-Pad9)
- J1 pad 90: Net-(J1-Pad90) -> unconnected-(J1-DO7-Pad90)
- J1 pad 91: Net-(J1-Pad91) -> unconnected-(J1-DI4-Pad91)
- J1 pad 92: Net-(J1-Pad92) -> unconnected-(J1-DI5-Pad92)
- J1 pad 93: Net-(J1-Pad93) -> unconnected-(J1-DI6-Pad93)
- J1 pad 94: Net-(J1-Pad94) -> unconnected-(J1-DI1-Pad94)
- J1 pad 95: Net-(J1-Pad95) -> unconnected-(J1-DI0-Pad95)
- J1 pad 96: Net-(J1-Pad96) -> unconnected-(J1-sINTA-Pad96)
- J1 pad 97: Net-(J1-Pad97) -> unconnected-(J1-~{sWO}-Pad97)
- J1 pad 98: Net-(J1-Pad98) -> unconnected-(J1-~{ERROR}-Pad98)
- J1 pad 99: Net-(J1-Pad99) -> unconnected-(J1-~{POC}-Pad99)
Other:
- board size 254 x 134.6 mm -> 254 x 137.8 mm
- net class Default removed
- rule pad_to_mask_clearance: 0.051 -> 0
- board text removed: "-"
