File: S-100-Template.kicad_pcb (KiCad board)
At the start: 2 copper layers, 254 x 137.8 mm, 3 parts

Commit message: Cleanup paste layer Add card ejector info
Parts:
- H1, H2: value MountingHole -> Card Ejector
