File: S-100-Template.kicad_pcb (KiCad board)
At the start: 2 copper layers, 254 x 137.8 mm, 3 parts

Commit message: Change size to to 5x10
Parts:
- added LOGO1: OSHW_Logo, Symbol:OSHW-Logo_11.4x12mm_SilkScreen, F.Cu at (264.2, 146.1)
- moved H1 3.17 mm to (25.4, 34.9)
- moved H2 3.17 mm to (266.7, 34.9)
Other:
- board size 254 x 137.8 mm -> 254 x 134.6 mm
